Commit message: lidar_camera added

File: catkin_ws/src/scout_ros/scout_description/urdf/mini.xacro (robot description, xacro)
@@ -97,3 +97,157 @@
     <!-- Gazebo definitions  -->
     <xacro:include filename="$(find scout_description)/urdf/scout_mini.gazebo" />
+    <link name="camera_link">
+        <visual>
+          <origin
+            xyz="0 0 01"
+            rpy="0 0 0" />
+            <geometry>
+              <box size="0.073000 0.276000 0.072000"/>
+            </geometry>
+        </visual>
+        <collision>
+          <origin
+            xyz="0 0 0"
+            rpy="0 0 0" />
+            <geometry>
+              <box size="0.073000 0.276000 0.072000"/>
+            </geometry>
+          </collision>
+        <inertial>
+          <origin
+            xyz="0 0 0"
+            rpy="0 0 0" />
+          <mass
+            value="0.1" />
+          <inertia
+            ixx="0.001E-10"
+            ixy="0.001E-10"
+            ixz="0.001E-10"
+            iyy="0.001E-10"
+            iyz="0.001E-10"
+            izz="0.001E-10" />
+        </inertial>
+      </link>
+    <joint name="camera_joint" type="fixed">
+        <origin
+          xyz="0.55 0 0"
+          rpy="0 0 0" />
+        <parent
+          link="base_link" />
+        <child
+          link="camera_link" />
+    </joint>
+    <gazebo reference="camera_link">
+        <sensor name="sensor_camera" type="depth">
+            <pose>0.0 0.0 0.0 0.0 0.0 0.0</pose>
+            <always_on>true</always_on>
+            <visualize>true</visualize>
+            <update_rate>10.0</update_rate>
+            <camera name="head">
+              <horizontal_fov>1.3962634</horizontal_fov>
+              <image>
+                  <width>640</width>
+                  <height>480</height>
+                  <format>R8G8B8</format>
+              </image>
+              <clip>
+                  <near>0.02</near>
+                  <far>300</far>
+              </clip>
+            </camera>
+            <plugin name="gazebo_ros_depth_camera_sensor" filename="libgazebo_ros_openni_kinect.so">
+              <baseline>0.2</baseline>
+              <alwaysOn>true</alwaysOn>
+              <!-- Keep this zero, update_rate in the parent <sensor> tag
+                will control the frame rate. -->
+              <updateRate>0.0</updateRate>
+              <cameraName>camera_ir</cameraName>
+              <imageTopicName>/limo/color/image_raw</imageTopicName>
+              <cameraInfoTopicName>/limo/color/camera_info</cameraInfoTopicName>
+              <depthImageTopicName>/limo/depth/image_raw</depthImageTopicName>
+              <depthImageCameraInfoTopicName>/limo/depth/camera_info</depthImageCameraInfoTopicName>
+              <pointCloudTopicName>/limo/depth/points</pointCloudTopicName>
+              <frameName>camera_link</frameName>
+              <cameraname>depth_camera_link</cameraname>
+              <pointCloudCutoff>0.5</pointCloudCutoff>
+              <pointCloudCutoffMax>3.0</pointCloudCutoffMax>
+              <distortionK1>0</distortionK1>
+              <distortionK2>0</distortionK2>
+              <distortionK3>0</distortionK3>
+              <distortionT1>0</distortionT1>
+              <distortionT2>0</distortionT2>
+              <CxPrime>0</CxPrime>
+              <Cx>0</Cx>
+              <Cy>0</Cy>
+              <focalLength>0</focalLength>
+              <hackBaseline>0</hackBaseline>
+            </plugin>
+        </sensor>
+    </gazebo>
+    <link name='laser_link'>
+        <pose>0 0 0 0 0 0</pose>
+        <inertial>
+            <mass value="0.1"/>
+            <origin xyz="0.0 0 0" rpy="0 0 0"/>
+            <inertia
+                ixx="1e-6" ixy="0" ixz="0"
+                iyy="1e-6" iyz="0"
+                izz="1e-6"
+            />
+        </inertial>
+        <visual name='laser_visual'>
+            <origin xyz="0 0 0" rpy="0 0 0"/>
+            <geometry>
+                <cylinder radius="0.02" length="0.01"/>
+            </geometry>
+        </visual>
+        <collision name='laser_collision'>
+            <origin xyz="0 0 0" rpy="0 0 0"/>
+            <geometry>
+                <cylinder radius="0.032" length="0.016"/>
+            </geometry>
+        </collision>
+      </link>
+      <joint
+    name="laser_joint"
+    type="fixed">
+    <origin
+      xyz="0.55 0 -0.1"
+      rpy="0 0 0" />
+    <parent
+      link="base_link" />
+    <child
+      link="laser_link" />
+  </joint>
+  <gazebo reference="laser_link">
+    <sensor type="ray" name="laser_sensor">
+      <pose>0 0 0 0 0 0</pose>
+      <visualize>false</visualize>
+      <update_rate>8</update_rate>
+      <ray>
+        <scan>
+          <horizontal>
+            <samples>720</samples>
+            <resolution>1</resolution>
+            <min_angle>-2.09439504</min_angle>
+            <max_angle>2.09439504</max_angle>
+          </horizontal>
+        </scan>
+        <range>
+          <min>0.05</min>
+          <max>8.0</max>
+          <resolution>0.01</resolution>
+        </range>
+        <noise>
+          <type>gaussian</type>
+          <mean>0.0</mean>
+          <stddev>0.01</stddev>
+        </noise>
+      </ray>
+      <plugin name="gazebo_ros_laser_sensor" filename="libgazebo_ros_laser.so">
+        <topicName>/robot1/scan</topicName>
+        <frameName>laser_link</frameName>
+      </plugin>
+    </sensor>
+  </gazebo>
 </robot>

Commit message: mini camera& lidar transparented

File: catkin_ws/src/scout_ros/scout_description/urdf/mini.xacro (robot description, xacro)
@@ -100,18 +100,13 @@
         <visual>
           <origin
-            xyz="0 0 01"
-            rpy="0 0 0" />
+            xyz="0.0 0 0.0"
+            rpy="0 0 3.141592" />
             <geometry>
-              <box size="0.073000 0.276000 0.072000"/>
+              <box size="0.035000 0.276000 0.05000"/>
             </geometry>
+            <material>
+                <color rgba="0.0 0.0 0.0 0.0"/>
+            </material>
         </visual>
-        <collision>
-          <origin
-            xyz="0 0 0"
-            rpy="0 0 0" />
-            <geometry>
-              <box size="0.073000 0.276000 0.072000"/>
-            </geometry>
-          </collision>
         <inertial>
           <origin
@@ -131,5 +126,5 @@
     <joint name="camera_joint" type="fixed">
         <origin
-          xyz="0.55 0 0"
+          xyz="0 0 0"
           rpy="0 0 0" />
         <parent
@@ -140,5 +135,5 @@
     <gazebo reference="camera_link">
         <sensor name="sensor_camera" type="depth">
-            <pose>0.0 0.0 0.0 0.0 0.0 0.0</pose>
+            <pose>0.3 0.0 0.0 0.0 0.0 0.0</pose>
             <always_on>true</always_on>
             <visualize>true</visualize>
@@ -163,9 +158,9 @@
               <updateRate>0.0</updateRate>
               <cameraName>camera_ir</cameraName>
-              <imageTopicName>/limo/color/image_raw</imageTopicName>
-              <cameraInfoTopicName>/limo/color/camera_info</cameraInfoTopicName>
-              <depthImageTopicName>/limo/depth/image_raw</depthImageTopicName>
-              <depthImageCameraInfoTopicName>/limo/depth/camera_info</depthImageCameraInfoTopicName>
-              <pointCloudTopicName>/limo/depth/points</pointCloudTopicName>
+              <imageTopicName>/camera/color/image_raw</imageTopicName>
+              <cameraInfoTopicName>/camera/color/camera_info</cameraInfoTopicName>
+              <depthImageTopicName>/camera/depth/image_raw</depthImageTopicName>
+              <depthImageCameraInfoTopicName>/camera/depth/camera_info</depthImageCameraInfoTopicName>
+              <pointCloudTopicName>/camera/depth/points</pointCloudTopicName>
               <frameName>camera_link</frameName>
               <cameraname>depth_camera_link</cameraname>
@@ -201,11 +196,8 @@
                 <cylinder radius="0.02" length="0.01"/>
             </geometry>
+            <material>
+                <color rgba="0.0 0.0 0.0 0.0"/>
+            </material>
         </visual>
-        <collision name='laser_collision'>
-            <origin xyz="0 0 0" rpy="0 0 0"/>
-            <geometry>
-                <cylinder radius="0.032" length="0.016"/>
-            </geometry>
-        </collision>
       </link>
       <joint

Commit message: camera complete

File: catkin_ws/src/scout_ros/scout_description/urdf/mini.xacro (robot description, xacro)
@@ -100,17 +100,26 @@
         <visual>
           <origin
-            xyz="0.0 0 0.0"
-            rpy="0 0 3.141592" />
-            <geometry>
-              <box size="0.035000 0.276000 0.05000"/>
-            </geometry>
-            <material>
-                <color rgba="0.0 0.0 0.0 0.0"/>
-            </material>
+            xyz="-0.32 0 0.0"
+            rpy="0 0 0" />
+            <geometry>
+              <box size="0.0073000 0.0276000 0.0072000"/>
+              <color rgba="1.0 0.0 0.0 1.0"/>
+            </geometry>
         </visual>
+        <collision>
+          <origin
+            xyz="0 0 0"
+            rpy="0 0 0" />
+            <geometry>
+              <box size="0.0073000 0.0276000 0.0072000"/>
+            </geometry>
+            <enabeled>false</enabeled>
+            <!-- collision falsed -->
+          </collision>
         <inertial>
           <origin
             xyz="0 0 0"
             rpy="0 0 0" />
+            <!-- mass를 무조건 줘야함 -->
           <mass
             value="0.1" />
@@ -126,5 +135,5 @@
     <joint name="camera_joint" type="fixed">
         <origin
-          xyz="0 0 0"
+          xyz="0.55 0 0"
           rpy="0 0 0" />
         <parent
@@ -135,5 +144,5 @@
     <gazebo reference="camera_link">
         <sensor name="sensor_camera" type="depth">
-            <pose>0.3 0.0 0.0 0.0 0.0 0.0</pose>
+            <pose>0.0 0.0 0.0 0.0 0.0 0.0</pose>
             <always_on>true</always_on>
             <visualize>true</visualize>
@@ -158,9 +167,9 @@
               <updateRate>0.0</updateRate>
               <cameraName>camera_ir</cameraName>
-              <imageTopicName>/camera/color/image_raw</imageTopicName>
-              <cameraInfoTopicName>/camera/color/camera_info</cameraInfoTopicName>
-              <depthImageTopicName>/camera/depth/image_raw</depthImageTopicName>
-              <depthImageCameraInfoTopicName>/camera/depth/camera_info</depthImageCameraInfoTopicName>
-              <pointCloudTopicName>/camera/depth/points</pointCloudTopicName>
+              <imageTopicName>/limo/color/image_raw</imageTopicName>
+              <cameraInfoTopicName>/limo/color/camera_info</cameraInfoTopicName>
+              <depthImageTopicName>/limo/depth/image_raw</depthImageTopicName>
+              <depthImageCameraInfoTopicName>/limo/depth/camera_info</depthImageCameraInfoTopicName>
+              <pointCloudTopicName>/limo/depth/points</pointCloudTopicName>
               <frameName>camera_link</frameName>
               <cameraname>depth_camera_link</cameraname>
@@ -196,8 +205,12 @@
                 <cylinder radius="0.02" length="0.01"/>
             </geometry>
-            <material>
-                <color rgba="0.0 0.0 0.0 0.0"/>
-            </material>
+            <color rgba="1.0 0.0 0.0 1.0"/>
         </visual>
+        <collision name='laser_collision'>
+            <origin xyz="0 0 0" rpy="0 0 0"/>
+            <geometry>
+                <cylinder radius="0.032" length="0.016"/>
+            </geometry>
+        </collision>
       </link>
       <joint

Commit message: front laser complete

File: catkin_ws/src/scout_ros/scout_description/urdf/mini.xacro (robot description, xacro)
@@ -167,9 +167,9 @@
               <updateRate>0.0</updateRate>
               <cameraName>camera_ir</cameraName>
-              <imageTopicName>/limo/color/image_raw</imageTopicName>
-              <cameraInfoTopicName>/limo/color/camera_info</cameraInfoTopicName>
-              <depthImageTopicName>/limo/depth/image_raw</depthImageTopicName>
-              <depthImageCameraInfoTopicName>/limo/depth/camera_info</depthImageCameraInfoTopicName>
-              <pointCloudTopicName>/limo/depth/points</pointCloudTopicName>
+              <imageTopicName>/camera/color/image_raw</imageTopicName>
+              <cameraInfoTopicName>/camera/color/camera_info</cameraInfoTopicName>
+              <depthImageTopicName>/camera/depth/image_raw</depthImageTopicName>
+              <depthImageCameraInfoTopicName>/camera/depth/camera_info</depthImageCameraInfoTopicName>
+              <pointCloudTopicName>/camera/depth/points</pointCloudTopicName>
               <frameName>camera_link</frameName>
               <cameraname>depth_camera_link</cameraname>
@@ -189,9 +189,9 @@
         </sensor>
     </gazebo>
-    <link name='laser_link'>
-        <pose>0 0 0 0 0 0</pose>
+    <link name='front_laser_link'>
+        <pose>0 0 0 0 0 0 0</pose>
         <inertial>
             <mass value="0.1"/>
-            <origin xyz="0.0 0 0" rpy="0 0 0"/>
+            <origin xyz="0.0 0 0.0" rpy="0 0 0"/>
             <inertia
                 ixx="1e-6" ixy="0" ixz="0"
@@ -201,31 +201,33 @@
         </inertial>
         <visual name='laser_visual'>
-            <origin xyz="0 0 0" rpy="0 0 0"/>
-            <geometry>
-                <cylinder radius="0.02" length="0.01"/>
-            </geometry>
-            <color rgba="1.0 0.0 0.0 1.0"/>
+            <origin xyz="0.0 0 -0.01" rpy="0 0 0"/>
+            <geometry>
+                <sphere radius="0.02" length="0.01"/>
+            </geometry>
+            <color rgba="1.0 0.0 0.0 0.0"/>
+            <enabeled>false</enabeled>
         </visual>
         <collision name='laser_collision'>
             <origin xyz="0 0 0" rpy="0 0 0"/>
             <geometry>
-                <cylinder radius="0.032" length="0.016"/>
-            </geometry>
+                <cylinder radius="0.0032" length="0.0016"/>
+            </geometry>
+            <enabeled>false</enabeled>
         </collision>
       </link>
-      <joint
+  <joint
     name="laser_joint"
     type="fixed">
     <origin
-      xyz="0.55 0 -0.1"
+      xyz="0.20 0 -0.020"
       rpy="0 0 0" />
     <parent
       link="base_link" />
     <child
-      link="laser_link" />
+      link="front_laser_link" />
   </joint>
-  <gazebo reference="laser_link">
+  <gazebo reference="front_laser_link">
     <sensor type="ray" name="laser_sensor">
-      <pose>0 0 0 0 0 0</pose>
+      <pose>0 0 0 0 0 0 0</pose>
       <visualize>false</visualize>
       <update_rate>8</update_rate>
@@ -251,6 +253,6 @@
       </ray>
       <plugin name="gazebo_ros_laser_sensor" filename="libgazebo_ros_laser.so">
-        <topicName>/robot1/scan</topicName>
-        <frameName>laser_link</frameName>
+        <topicName>/scan/front</topicName>
+        <frameName>front_laser_link</frameName>
       </plugin>
     </sensor>

Commit message: scout gazebo front lidar update

File: catkin_ws/src/scout_ros/scout_description/urdf/mini.xacro (robot description, xacro)
@@ -200,16 +200,15 @@
             />
         </inertial>
-        <visual name='laser_visual'>
+        <visual name='front_laser_visual'>
             <origin xyz="0.0 0 -0.01" rpy="0 0 0"/>
             <geometry>
-                <sphere radius="0.02" length="0.01"/>
-            </geometry>
-            <color rgba="1.0 0.0 0.0 0.0"/>
-            <enabeled>false</enabeled>
+                <sphere radius="0.002"/>
+            </geometry>
+            <color rgba="0.0 0.0 0.0 0.0"/>
         </visual>
-        <collision name='laser_collision'>
+        <collision name='front_laser_collision'>
             <origin xyz="0 0 0" rpy="0 0 0"/>
             <geometry>
-                <cylinder radius="0.0032" length="0.0016"/>
+                <sphere radius="0.002"/>
             </geometry>
             <enabeled>false</enabeled>
@@ -217,5 +216,5 @@
       </link>
   <joint
-    name="laser_joint"
+    name="front_laser_joint"
     type="fixed">
     <origin
@@ -258,3 +257,72 @@
     </sensor>
   </gazebo>
+<!-- back laser -->
+  <link name='back_laser_link'>
+    <pose>0 0 0 0 0 0 </pose>
+    <inertial>
+        <mass value="0.1"/>
+        <origin xyz="0.0 0 0.0" rpy="0 0 0"/>
+        <inertia
+            ixx="1e-6" ixy="0" ixz="0"
+            iyy="1e-6" iyz="0"
+            izz="1e-6"
+        />
+    </inertial>
+    <visual name='laser_visual'>
+        <origin xyz="0.0 0 0" rpy="0 0 0"/>
+        <geometry>
+            <sphere radius="0.002"/>
+        </geometry>
+        <color rgba="1.0 0.0 0.0 0.0"/>
+    </visual>
+    <collision name='laser_collision'>
+        <origin xyz="0 0 0" rpy="0 0 0"/>
+        <geometry>
+            <sphere radius="0.002"/>
+        </geometry>
+        <enabeled>false</enabeled>
+    </collision>
+  </link>
+  <joint
+    name="back_laser_joint"
+    type="fixed">
+    <origin
+      xyz="-0.30 0 0.15"
+      rpy="0 0 -3.141592" />
+    <parent
+      link="base_link" />
+    <child
+      link="back_laser_link" />
+  </joint>
+  <gazebo reference="back_laser_link">
+    <sensor type="ray" name="laser_sensor">
+      <pose>0 0 0 0 0 0</pose>
+      <visualize>false</visualize>
+      <update_rate>8</update_rate>
+      <ray>
+        <scan>
+          <horizontal>
+            <samples>720</samples>
+            <resolution>1</resolution>
+            <min_angle>2.09439504</min_angle>
+            <max_angle>-2.09439504</max_angle>
+          </horizontal>
+        </scan>
+        <range>
+          <min>0.50</min>
+          <max>8.0</max>
+          <resolution>0.01</resolution>
+        </range>
+        <noise>
+          <type>gaussian</type>
+          <mean>0.0</mean>
+          <stddev>0.01</stddev>
+        </noise>
+      </ray>
+      <plugin name="gazebo_ros_laser_sensor" filename="libgazebo_ros_laser.so">
+        <topicName>/scan/back</topicName>
+        <frameName>back_laser_link</frameName>
+      </plugin>
+    </sensor>
+  </gazebo>
 </robot>
